File: keebwirdv1.kicad_pcb (KiCad board)
At the start: 2 copper layers, 258 x 110 mm, 69 parts, among them U0 ProMicro

Commit message: keebwird.kicad_pcb
Parts:
- added SW1: SW_Push, keebwird:ResetSW_1side, F.Cu at (192.7, 54.9)
- D0, D1, D10, D11, D12, D13, D14, D15, D16, D17, D18, D19, D2, D20, D21, D22, D23, D24, D25, D26, D27, D28, D29, D3, D30, D31, D32, D33, D4, D5, D6, D7, D8, D9: footprint Keebio-Parts:Diode -> keebwird:Diode
- MX0, MX1, MX10, MX11, MX12, MX13, MX14, MX15, MX16, MX17, MX18, MX19, MX2, MX20, MX21, MX22, MX23, MX24, MX25, MX26, MX27, MX28, MX29, MX3, MX30, MX31, MX32, MX33, MX4, MX6, MX7, MX8, MX9: footprint Kailh_Choc:KailhChoc-1U -> keebwird:KailhChoc-1U
- MX5: renamed from MXe; footprint Kailh_Choc:KailhChoc-1U -> keebwird:KailhChoc-1U
- U0: footprint Keebio-Parts:ArduinoProMicro -> keebwird:ArduinoProMicro
Connections:
- U0 pad 3: Net-(U0-Pad3) -> GND
- U0 pad 4: Net-(U0-Pad4) -> GND
Routing:
- net Net-(SW1-Pad1): track 0.00 -> 49.4 mm
- added copper zone on B.Cu, net GND
- added copper zone on F.Cu, net GND
Other:
- board size 258 x 110 mm -> 248.1 x 107.5 mm
